File: X60.sch (KiCad schematic (older format))
At the start: 21 parts, among them SW1 SW_Push, U1 ATmega32U4-MU, U2 PRTR5V0U2X, Y1 16MHz

Commit message: X60
Parts:
- removed L1: 60R@100MHz, Inductor_SMD:L_1206_3216Metric, symbol Device:L_Core_Ferrite_Small
- removed U1: ATmega32U4-MU, Package_DFN_QFN:QFN-44-1EP_7x7mm_P0.5mm_EP5.2x5.2mm, symbol MCU_Microchip_ATmega:ATmega32U4-MU
- removed U2: PRTR5V0U2X, random-keyboard-parts:SOT143B, symbol ai03-locallib:PRTR5V0U2X
- added U1: ATmega32U4-AU, Package_QFP:TQFP-44_10x10mm_P0.8mm, symbol MCU_Microchip_ATmega:ATmega32U4-AU
- C1, C2, C3, C4, C5, C6, C7: footprint Capacitor_SMD:C_0603_1608Metric -> Capacitor_SMD:C_0603_1608Metric_Pad1.08x0.95mm_HandSolder
- R1, R2, R3, R4, R5, R6: footprint Resistor_SMD:R_0603_1608Metric -> Resistor_SMD:R_0603_1608Metric_Pad0.98x0.95mm_HandSolder
Connections:
- wire segments 70 -> 66
Changed lines of the file:
@@
 EESchema Schematic File Version 4
-LIBS:JIS60-cache
 EELAYER 30 0
 EELAYER END
@@
 F 0 "C1" H 4017 7121 50  0000 L CNN
 F 1 "0.1uF" H 4017 7030 50  0000 L CNN
-F 2 "Capacitor_SMD:C_0603_1608Metric" H 3925 7075 50  0001 C CNN
+F 2 "Capacitor_SMD:C_0603_1608Metric_Pad1.08x0.95mm_HandSolder" H 3925 7075 50  0001 C CNN
 F 3 "~" H 3925 7075 50  0001 C CNN
 	1    3925 7075
@@
 F 0 "C2" H 4392 7121 50  0000 L CNN
 F 1 "0.1uF" H 4392 7030 50  0000 L CNN
-F 2 "Capacitor_SMD:C_0603_1608Metric" H 4300 7075 50  0001 C CNN
+F 2 "Capacitor_SMD:C_0603_1608Metric_Pad1.08x0.95mm_HandSolder" H 4300 7075 50  0001 C CNN
 F 3 "~" H 4300 7075 50  0001 C CNN
 	1    4300 7075
@@
 F 0 "C3" H 4767 7121 50  0000 L CNN
 F 1 "0.1uF" H 4767 7030 50  0000 L CNN
-F 2 "Capacitor_SMD:C_0603_1608Metric" H 4675 7075 50  0001 C CNN
+F 2 "Capacitor_SMD:C_0603_1608Metric_Pad1.08x0.95mm_HandSolder" H 4675 7075 50  0001 C CNN
 F 3 "~" H 4675 7075 50  0001 C CNN
 	1    4675 7075
@@
 F 0 "C4" H 5142 7121 50  0000 L CNN
 F 1 "10uF" H 5142 7030 50  0000 L CNN
-F 2 "Capacitor_SMD:C_0603_1608Metric" H 5050 7075 50  0001 C CNN
+F 2 "Capacitor_SMD:C_0603_1608Metric_Pad1.08x0.95mm_HandSolder" H 5050 7075 50  0001 C CNN
 F 3 "~" H 5050 7075 50  0001 C CNN
 	1    5050 7075
@@
 F 0 "C5" H 1217 4146 50  0000 L CNN
 F 1 "22pF" H 1217 4055 50  0000 L CNN
-F 2 "Capacitor_SMD:C_0603_1608Metric" H 1125 4100 50  0001 C CNN
+F 2 "Capacitor_SMD:C_0603_1608Metric_Pad1.08x0.95mm_HandSolder" H 1125 4100 50  0001 C CNN
 F 3 "~" H 1125 4100 50  0001 C CNN
 	1    1125 4100
@@
 F 0 "C6" H 1217 4346 50  0000 L CNN
 F 1 "22pF" H 1217 4255 50  0000 L CNN
-F 2 "Capacitor_SMD:C_0603_1608Metric" H 1125 4300 50  0001 C CNN
+F 2 "Capacitor_SMD:C_0603_1608Metric_Pad1.08x0.95mm_HandSolder" H 1125 4300 50  0001 C CNN
 F 3 "~" H 1125 4300 50  0001 C CNN
 	1    1125 4300
@@
 F 0 "R1" V 1304 4900 50  0000 C CNN
 F 1 "22" V 1395 4900 50  0000 C CNN
-F 2 "Resistor_SMD:R_0603_1608Metric" H 1500 4900 50  0001 C CNN
+F 2 "Resistor_SMD:R_0603_1608Metric_Pad0.98x0.95mm_HandSolder" H 1500 4900 50  0001 C CNN
 F 3 "~" H 1500 4900 50  0001 C CNN
 	1    1500 4900
@@
 F 0 "R3" V 1304 5000 50  0000 C CNN
 F 1 "22" V 1395 5000 50  0000 C CNN
-F 2 "Resistor_SMD:R_0603_1608Metric" H 1500 5000 50  0001 C CNN
+F 2 "Resistor_SMD:R_0603_1608Metric_Pad0.98x0.95mm_HandSolder" H 1500 5000 50  0001 C CNN
 F 3 "~" H 1500 5000 50  0001 C CNN
 	1    1500 5000
@@
 F 0 "C7" H 1717 5346 50  0000 L CNN
 F 1 "1uF" H 1717 5255 50  0000 L CNN
-F 2 "Capacitor_SMD:C_0603_1608Metric" H 1625 5300 50  0001 C CNN
+F 2 "Capacitor_SMD:C_0603_1608Metric_Pad1.08x0.95mm_HandSolder" H 1625 5300 50  0001 C CNN
 F 3 "~" H 1625 5300 50  0001 C CNN
 	1    1625 5300
@@
 F 0 "R4" V 3354 6000 50  0000 C CNN
 F 1 "1k" V 3445 6000 50  0000 C CNN
-F 2 "Resistor_SMD:R_0603_1608Metric" H 3550 6000 50  0001 C CNN
+F 2 "Resistor_SMD:R_0603_1608Metric_Pad0.98x0.95mm_HandSolder" H 3550 6000 50  0001 C CNN
 F 3 "~" H 3550 6000 50  0001 C CNN
 	1    3550 6000
@@
 	1    0    0    -1
 $EndComp
-Wire Wire Line
-	2300 3600 2400 3600
-Wire Wire Line
-	1975 7200 2300 7200
-$Comp
-L MCU_Microchip_ATmega:ATmega32U4-MU U1
-U 1 1 5FC739A7
-P 2400 5400
-F 0 "U1" H 2400 3511 50  0000 C CNN
-F 1 "ATmega32U4-MU" H 2400 3420 50  0000 C CNN
-F 2 "Package_DFN_QFN:QFN-44-1EP_7x7mm_P0.5mm_EP5.2x5.2mm" H 2400 5400 50  0001 C CIN
-F 3 "http://ww1.microchip.com/downloads/en/DeviceDoc/Atmel-7766-8-bit-AVR-ATmega16U4-32U4_Datasheet.pdf" H 2400 5400 50  0001 C CNN
-	1    2400 5400
-	1    0    0    -1
-$EndComp
-Connection ~ 2300 3600
-Wire Wire Line
-	2400 7200 2300 7200
-Connection ~ 2300 7200
-Wire Wire Line
-	2500 3600 2400 3600
-Connection ~ 2400 3600
 $Comp
 L Switch:SW_Push SW1
@@
 F 0 "R5" H 1591 3629 50  0000 R CNN
 F 1 "10k" H 1591 3720 50  0000 R CNN
-F 2 "Resistor_SMD:R_0603_1608Metric" H 1650 3675 50  0001 C CNN
+F 2 "Resistor_SMD:R_0603_1608Metric_Pad0.98x0.95mm_HandSolder" H 1650 3675 50  0001 C CNN
 F 3 "~" H 1650 3675 50  0001 C CNN
 	1    1650 3675
@@
 F 3 "" H 1800 1675 60  0001 C CNN
 	1    1800 1675
-	1    0    0    -1
-$EndComp
-$Comp
-L ai03-locallib:PRTR5V0U2X U2
-U 1 1 60F0A61D
-P 3900 2450
-F 0 "U2" H 3900 2747 60  0000 C CNN
-F 1 "PRTR5V0U2X" H 3900 2641 60  0000 C CNN
-F 2 "random-keyboard-parts:SOT143B" H 3900 2450 60  0001 C CNN
-F 3 "" H 3900 2450 60  0001 C CNN
-	1    3900 2450
 	1    0    0    -1
 $EndComp
@@
 F 0 "R2" H 2316 2379 50  0000 R CNN
 F 1 "5.1k" H 2316 2470 50  0000 R CNN
-F 2 "Resistor_SMD:R_0603_1608Metric" H 2375 2425 50  0001 C CNN
+F 2 "Resistor_SMD:R_0603_1608Metric_Pad0.98x0.95mm_HandSolder" H 2375 2425 50  0001 C CNN
 F 3 "~" H 2375 2425 50  0001 C CNN
 	1    2375 2425
@@
 F 0 "R6" H 2616 2379 50  0000 R CNN
 F 1 "5.1k" H 2616 2470 50  0000 R CNN
-F 2 "Resistor_SMD:R_0603_1608Metric" H 2675 2425 50  0001 C CNN
+F 2 "Resistor_SMD:R_0603_1608Metric_Pad0.98x0.95mm_HandSolder" H 2675 2425 50  0001 C CNN
 F 3 "~" H 2675 2425 50  0001 C CNN
 	1    2675 2425
@@
 	2375 2600 2375 2525
 Connection ~ 2525 2600
-$Comp
-L power:GND #PWR0116
-U 1 1 60F2B593
-P 3250 2400
-F 0 "#PWR0116" H 3250 2150 50  0001 C CNN
-F 1 "GND" H 3255 2227 50  0000 C CNN
-F 2 "" H 3250 2400 50  0001 C CNN
-F 3 "" H 3250 2400 50  0001 C CNN
-	1    3250 2400
-	1    0    0    -1
-$EndComp
-Wire Wire Line
-	3250 2400 3600 2400
-Text GLabel 3600 2700 0    60   Input ~ 0
-D+
-Text GLabel 4200 2700 2    60   Input ~ 0
-D-
-Wire Wire Line
-	4200 2700 4200 2500
-Wire Wire Line
-	3600 2700 3600 2500
-$Comp
-L power:VCC #PWR0117
-U 1 1 60F35AAD
-P 4325 2400
-F 0 "#PWR0117" H 4325 2250 50  0001 C CNN
-F 1 "VCC" H 4342 2573 50  0000 C CNN
-F 2 "" H 4325 2400 50  0001 C CNN
-F 3 "" H 4325 2400 50  0001 C CNN
-	1    4325 2400
-	1    0    0    -1
-$EndComp
-Wire Wire Line
-	4325 2400 4200 2400
-$Comp
-L Device:L_Core_Ferrite_Small L1
-U 1 1 60F78093
-P 4625 1900
-F 0 "L1" V 4830 1900 50  0000 C CNN
-F 1 "60R@100MHz" V 4739 1900 50  0000 C CNN
-F 2 "Inductor_SMD:L_1206_3216Metric" H 4625 1900 50  0001 C CNN
-F 3 "~" H 4625 1900 50  0001 C CNN
-	1    4625 1900
-	0    -1   -1   0
-$EndComp
 NoConn ~ 1900 1325
 NoConn ~ 1900 1925
-$Comp
-L power:Earth #PWR0118
-U 1 1 60F7C40D
-P 4525 1900
-F 0 "#PWR0118" H 4525 1650 50  0001 C CNN
-F 1 "Earth" H 4525 1750 50  0001 C CNN
-F 2 "" H 4525 1900 50  0001 C CNN
-F 3 "~" H 4525 1900 50  0001 C CNN
-	1    4525 1900
-	1    0    0    -1
-$EndComp
-$Comp
-L power:GND #PWR0119
-U 1 1 60F83785
-P 4725 1900
-F 0 "#PWR0119" H 4725 1650 50  0001 C CNN
-F 1 "GND" H 4730 1727 50  0000 C CNN
-F 2 "" H 4725 1900 50  0001 C CNN
-F 3 "" H 4725 1900 50  0001 C CNN
-	1    4725 1900
-	1    0    0    -1
-$EndComp
 $Comp
 L Device:D_TVS D32
@@
 Text GLabel 3000 4800 2    60   Input ~ 0
 COL6
+$Comp
+L MCU_Microchip_ATmega:ATmega32U4-AU U1
+U 1 1 61473023
+P 2400 5400
+F 0 "U1" H 2400 3511 50  0000 C CNN
+F 1 "ATmega32U4-AU" H 2400 3420 50  0000 C CNN
+F 2 "Package_QFP:TQFP-44_10x10mm_P0.8mm" H 2400 5400 50  0001 C CIN
+F 3 "http://ww1.microchip.com/downloads/en/DeviceDoc/Atmel-7766-8-bit-AVR-ATmega16U4-32U4_Datasheet.pdf" H 2400 5400 50  0001 C CNN
+	1    2400 5400
+	1    0    0    -1
+$EndComp
+Connection ~ 2400 3600
+Connection ~ 2300 7200
+Connection ~ 2300 3600
+Wire Wire Line
+	2400 7200 2300 7200
+Wire Wire Line
+	1975 7200 2300 7200
+Wire Wire Line
+	2500 3600 2400 3600
+Wire Wire Line
+	2300 3600 2400 3600
 $EndSCHEMATC
