File: matrix.sch (KiCad schematic (older format))
At the start: 129 parts

Commit message: X60
Parts:
- added D37: SOD-123, Diode_SMD:D_SOD-123, symbol Device:D_Small
- K_ENTER1: footprint MX_Only:MXOnly-ISO-ROTATED-Hotswap -> MX_Only:MXOnly-2.25U-Hotswap-ReversedStabilizers
- K_LALT1, K_LGUI1, K_SPC2, K_]1: footprint MX_Only:MXOnly-1U-Hotswap -> MX_Only:MXOnly-1.5U-Hotswap
- K_LSFT1: footprint MX_Only:MXOnly-2.25U-Hotswap -> MX_Only:MXOnly-1.5U-Hotswap
- K_NFER1: footprint MX_Only:MXOnly-1.25U-Hotswap -> MX_Only:MXOnly-2.75U-Hotswap-ReversedStabilizers
- K_RCTRL1: footprint MX_Only:MXOnly-1.25U-Hotswap -> MX_Only:MXOnly-1U-Hotswap
- K_SPC1: footprint MX_Only:MXOnly-6U-Centered-Hotswap-ReversedStabilizers -> MX_Only:MXOnly-2.25U-Hotswap-ReversedStabilizers
- K_SRSFT2: footprint MX_Only:MXOnly-1.75U-Hotswap -> MX_Only:MXOnly-1U-Hotswap
Connections:
- net COL1: now also K_Z1.1 (COL)
- net COL10: now also K_/1.1 (COL); no longer K_.1.1 (COL)
- net COL11: now also K_SRSFT1.1 (COL); no longer K_/1.1 (COL)
- net COL12: now also K_ENTER1.1 (COL), K_\1.1 (COL); no longer K_SBSPC2.1 (COL), K_SRSFT1.1 (COL)
- net COL13: now also K_SBSPC2.1 (COL); no longer K_ENTER1.1 (COL), K_\1.1 (COL)
- net COL2: now also K_X1.1 (COL); no longer K_Z1.1 (COL)
- net COL3: now also K_C1.1 (COL); no longer K_NFER1.1 (COL), K_X1.1 (COL)
- net COL4: now also K_NFER1.1 (COL), K_V1.1 (COL); no longer K_C1.1 (COL)
- net COL5: now also K_B1.1 (COL); no longer K_V1.1 (COL)
- net COL6: now also K_N1.1 (COL); no longer K_B1.1 (COL)
- net COL7: now also K_M1.1 (COL); no longer K_N1.1 (COL), K_SPC2.2 (ROW)
- net COL8: now also K_,1.1 (COL); no longer K_M1.1 (COL)
- net COL9: now also K_.1.1 (COL), K_SPC2.1 (COL); no longer K_,1.1 (COL)
- net ROW1: now also D17.1 (K); no longer D71.1 (K)
- net ROW2: no longer D17.1 (K)
- net ROW3: now also D71.1 (K)
- net ROW4: now also D37.1 (K)
- net at D42.2 (A), K_SPC1.2 (ROW): no longer K_SPC2.1 (COL)
- new net: D37.2 (A), K_SPC2.2 (ROW)
Other:
- moved on the sheet: D1, D15, D17, D21, D22, D26, D31, D36, D41, D47, D52, D57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
